Commit message: updated path references

File: scara_robot/models/params_macro.xacro (robot description, xacro)
@@ -3,5 +3,5 @@
     <!-- \\\ Load YAML Files \\\ -->
     <!--Declare the name of yaml file-->
-    <xacro:property name="yaml_file" value="$(find scara)/config/scara_params.yaml"/>
+    <xacro:property name="yaml_file" value="$(find scara_robot)/config/scara_params.yaml"/>
     <!--Load the parameters in a dictionary called "props"-->
     <xacro:property name="props" value="${xacro.load_yaml(yaml_file)}"/>

File: scara_robot/models/scara_robot.xacro (robot description, xacro)
@@ -3,5 +3,5 @@
     <!-- \\\\\\ Build 2DoF Arm Robot \\\\\\ -->
     <!-- \\\ Include Parameters and Macros \\\ -->
-    <xacro:include filename="$(find scara)/models/params_macro.xacro"/>
+    <xacro:include filename="$(find scara_robot)/models/params_macro.xacro"/>
     <!-- Chassis Link: Fictitious Link -->
     <link name = "world"/>

Commit message: added mesh & solved package issue

File: scara_robot/models/params_macro.xacro (robot description, xacro)
@@ -81,4 +81,41 @@
         </gazebo>
     </xacro:macro>
+    <!--SCARA ARM-->
+    <xacro:macro name="scara_arm" params="name x:=0 y:=0 z:=0 phi:=0 theta:=0 psi:=0 scale_x:=1 scale_y:=1 scale_z:=1 mass:=1 cogx:=0 cogy:=0 cogz:=0 colour:=White">
+        <link name="${name}">
+            <!--Visual-->
+            <visual>
+                <!--Origin tag is the pose of Center of Mass-->
+                <origin xyz="${x} ${y} ${z}" rpy="${phi} ${theta} ${psi}" />
+                <geometry>
+                    <mesh filename = "$(find scara_robot)/meshes/arm_model.stl" scale = "${scale_x} ${scale_y} ${scale_z}"/>
+                </geometry>
+            </visual>
+            <!--Collision: same as Visual-->
+            <collision>
+                <origin xyz="${x} ${y} ${z}" rpy="${phi} ${theta} ${psi}" />
+                <geometry>
+                    <mesh filename = "$(find scara_robot)/meshes/arm_model.stl" scale = "${scale_x} ${scale_y} ${scale_z}"/>
+                </geometry>
+            </collision>
+            <!--Inertial Tensor-->
+            <inertial>
+                <mass value = "3.84886936" />
+                <inertia ixx = "0.00680632" ixy = "0" ixz = "0" iyy = "0.03365825" iyz = "0" izz = "0.03989022"/>
+                <origin xyz="${x} ${y} ${z}" rpy="${phi} ${theta} ${psi}" />
+            </inertial>
+        </link>
+        <!-- Gazebo simulation settings -->
+        <gazebo reference="${name}">
+            <selfCollide>true</selfCollide>
+            <static>false</static>
+            <turnGravityOff>false</turnGravityOff>
+            <kp>1000000.0</kp>
+            <kd>1.0</kd>
+            <mu1>0.8</mu1>
+            <mu2>0.8</mu2>
+            <material>Gazebo/${colour}</material>
+        </gazebo>
+    </xacro:macro>
     <!--Transmission Block-->
     <xacro:macro name="transmission_block" params="joint_name location Type:=Position">

File: scara_robot/models/scara_robot.xacro (robot description, xacro)
@@ -15,5 +15,5 @@
                             mass="${m_base}" colour="Black"/>
     <!--Arm 1-->
-    <xacro:cylinder_link name="arm1" length="${a1}" radius="${r1}"
+    <xacro:scara_arm name="arm1" scale_x="1.5"
                             z="${a1/2}" mass="${m1}" colour="White"
                             cogz="${a1/2}"/>
@@ -27,6 +27,5 @@
     </joint>
     <!--Arm 2-->
-    <xacro:cylinder_link name="arm2" length="${a2}" radius="${r2}"
-                            z="${a2/2}" mass="${m2}" colour="Red"
+    <xacro:scara_arm name="arm2" z="${a2/2}" mass="${m2}" colour="Red"
                             cogz="${a2/2}"/>
     <!-- Joint 2-->
@@ -60,5 +59,5 @@
     <gazebo>
         <plugin name="gazebo_ros_control" filename="libgazebo_ros_control.so">
-            <robotNamespace>/scara</robotNamespace>
+            <robotNamespace>/scara_robot</robotNamespace>
         </plugin>
     </gazebo>

Commit message: added kinematic control and solved modelling issues

File: scara_robot/models/params_macro.xacro (robot description, xacro)
@@ -30,4 +30,5 @@
     <xacro:property name="base_width" value="${props['kinematic_params']['base_width']}"/>
     <xacro:property name="base_height" value="${props['kinematic_params']['base_height']}"/>
+    <xacro:property name="arm_height" value="${props['kinematic_params']['arm_height']}"/>
     <!-- \\\ Sensor Data \\\ -->
     <xacro:property name="imu_mass" value="${props['imu']['mass']}"/>
@@ -73,5 +74,5 @@
             <selfCollide>true</selfCollide>
             <static>false</static>
-            <turnGravityOff>false</turnGravityOff>
+            <turnGravityOff>true</turnGravityOff>
             <kp>1000000.0</kp>
             <kd>1.0</kd>

File: scara_robot/models/scara_robot.xacro (robot description, xacro)
@@ -15,10 +15,8 @@
                             mass="${m_base}" colour="Black"/>
     <!--Arm 1-->
-    <xacro:scara_arm name="arm1" scale_x="1.8"
-                            z="${a1/2}" mass="${m1}" colour="White"
-                            cogz="${a1/2}"/>
+    <xacro:scara_arm name="arm1" scale_x="1.8" mass="${m1}" colour="White"/>
     <!-- Joint 1-->
     <joint name="joint_1" type="revolute">
-        <origin xyz="0 0 0" rpy="0 0 0"/>
+        <origin xyz="0 0 ${base_height/2}" rpy="0 0 0"/>
         <parent link="base"/>
         <child link="arm1"/>
@@ -27,26 +25,24 @@
     </joint>
     <!--Arm 2-->
-    <xacro:scara_arm name="arm2" z="${a2/2}" mass="${m2}" colour="Red"
-                            cogz="${a2/2}"/>
+    <xacro:scara_arm name="arm2" mass="${m2}" colour="Red"/>
     <!-- Joint 2-->
     <joint name="joint_2" type="revolute">
-        <origin xyz="0.4 0 0.03" rpy="0 0 0"/>
+        <origin xyz="0.4 0 ${arm_height}" rpy="0 0 0"/>
         <parent link="arm1"/>
         <child link="arm2"/>
         <axis xyz="0 0 1"/>
-        <limit effort="${joint_effort}" velocity="${joint_vel}" lower="0.0" upper="0.0"/>
+        <limit effort="${joint_effort}" velocity="${joint_vel}" lower="${-joint_limit}" upper="${joint_limit}"/>
         <dynamics damping="0.0"/>
     </joint>
     <!--Linear needle-->
-    <xacro:cylinder_link name="lin" length="${a3}" radius="${r3}"
-                            z="${a3/2}" mass="${m3}" colour="Green"
-                            cogz="${a3/2}"/>
+    <xacro:cylinder_link name="lin" length="${(base_height + 2*arm_height)}" radius="${r3}" z="${(base_height + 2*arm_height)/2}"
+                            mass="${m3}" colour="Green"/>
     <!-- Joint 3 (linear)-->
     <joint name="joint_3" type="prismatic">
-    <origin xyz="0.25 0 ${a3/2}" rpy="0 0 0"/>
+    <origin xyz="0.25 0 ${-(base_height + arm_height)}" rpy="0 0 0"/>
     <parent link="arm2"/>
     <child link="lin"/>
     <axis xyz="0 0 1"/>
-    <limit effort="${joint_effort}" velocity="${joint_vel}" lower="${-a3/2}" upper="${a3/2}"/>
+    <limit effort="${joint_effort}" velocity="${joint_vel}" lower="0" upper="${(base_height + arm_height)}"/>
     <dynamics damping="0.0"/>
     </joint>

Commit message: parameterized inertia for scara arm

File: scara_robot/models/params_macro.xacro (robot description, xacro)
@@ -30,5 +30,8 @@
     <xacro:property name="base_width" value="${props['kinematic_params']['base_width']}"/>
     <xacro:property name="base_height" value="${props['kinematic_params']['base_height']}"/>
+    <!-- Params of scara_arm-->
     <xacro:property name="arm_height" value="${props['kinematic_params']['arm_height']}"/>
+    <xacro:property name="arm_width" value="${props['kinematic_params']['arm_width']}"/>
+    <xacro:property name="arm_length" value="${props['kinematic_params']['arm_length']}"/>
     <!-- \\\ Sensor Data \\\ -->
     <xacro:property name="imu_mass" value="${props['imu']['mass']}"/>
@@ -46,4 +49,14 @@
             <inertia ixx="${mass/12*(3*radius*radius + length*length) + mass*length*length/4}" ixy="0.0" ixz="0.0"
                          iyy="${mass/12*(3*radius*radius + length*length) + mass*length*length/4}" iyz="0.0" izz="${mass*radius*radius/2}"/>
+            <origin xyz="${cogx} ${cogy} ${cogz}" rpy="0 0 0"/>
+        </inertial>
+    </xacro:macro>
+    <!-- Inertial Matrix of Scara Arm
+    simplified as rectangular plate -->
+    <xacro:macro name="inertial_matrix_arm" params="mass length_x width_y height_z cogx:=0 cogy:=0 cogz:=0">
+        <inertial>
+            <mass value="${mass}"/>
+            <inertia ixx="${mass/12*(width_y*width_y + height_z*height_z)}" ixy="0.0" ixz="0.0"
+                         iyy="${mass/12*(length_x*length_x + height_z*height_z)}" iyz="0.0" izz="${mass/12*(length_x*length_x + width_y*width_y)}"/>
             <origin xyz="${cogx} ${cogy} ${cogz}" rpy="0 0 0"/>
         </inertial>
@@ -101,9 +114,5 @@
             </collision>
             <!--Inertial Tensor-->
-            <inertial>
-                <mass value = "3.84886936" />
-                <inertia ixx = "0.00680632" ixy = "0" ixz = "0" iyy = "0.03365825" iyz = "0" izz = "0.03989022"/>
-                <origin xyz="${x} ${y} ${z}" rpy="${phi} ${theta} ${psi}" />
-            </inertial>
+            <xacro:inertial_matrix_arm mass="${mass}" length_x="${arm_length*scale_x}" width_y="${arm_width*scale_y}" height_z="${arm_height*scale_z}" cogx="${cogx}" cogy="${cogy}" cogz="${cogz}"/>
         </link>
         <!-- Gazebo simulation settings -->

File: scara_robot/models/scara_robot.xacro (robot description, xacro)
@@ -38,5 +38,6 @@
     <xacro:cylinder_link name="lin" length="${(base_height + 2*arm_height)}" radius="${r3}" z="${(base_height + 2*arm_height)/2}"
                             mass="${m3}" colour="Green"/>
-    <!-- Joint 3 (linear)-->
+    <!-- Joint 3 (linear)
+        origon of joint set to ZERO, therefore controller input equals absolute z-position -->
     <joint name="joint_3" type="prismatic">
     <origin xyz="0.25 0 ${-(base_height + arm_height)}" rpy="0 0 0"/>

Commit message: changed joint1 & parameterized scale

File: scara_robot/models/params_macro.xacro (robot description, xacro)
@@ -34,4 +34,7 @@
     <xacro:property name="arm_width" value="${props['kinematic_params']['arm_width']}"/>
     <xacro:property name="arm_length" value="${props['kinematic_params']['arm_length']}"/>
+    <xacro:property name="arm_dist_rot" value="${props['kinematic_params']['arm_dist_rot']}"/>
+    <xacro:property name="scalex_1" value="${props['kinematic_params']['scalex_1']}"/>
+    <xacro:property name="scalex_2" value="${props['kinematic_params']['scalex_2']}"/>
     <!-- \\\ Sensor Data \\\ -->
     <xacro:property name="imu_mass" value="${props['imu']['mass']}"/>

File: scara_robot/models/scara_robot.xacro (robot description, xacro)
@@ -15,18 +15,18 @@
                             mass="${m_base}" colour="Black"/>
     <!--Arm 1-->
-    <xacro:scara_arm name="arm1" scale_x="1.8" mass="${m1}" colour="White"/>
+    <xacro:scara_arm name="arm1" scale_x="${scalex_1}" mass="${m1}" colour="White"/>
     <!-- Joint 1-->
-    <joint name="joint_1" type="revolute">
+    <joint name="joint_1" type="continuous">
         <origin xyz="0 0 ${base_height/2}" rpy="0 0 0"/>
         <parent link="base"/>
         <child link="arm1"/>
         <axis xyz="0 0 1"/>
-        <limit effort="${joint_effort}" velocity="${joint_vel}" lower="${-joint_limit}" upper="${joint_limit}"/>
+        <limit effort="${joint_effort}" velocity="${joint_vel}"/>
     </joint>
     <!--Arm 2-->
-    <xacro:scara_arm name="arm2" mass="${m2}" colour="Red"/>
+    <xacro:scara_arm name="arm2" scale_x="${scalex_2}" mass="${m2}" colour="Red"/>
     <!-- Joint 2-->
     <joint name="joint_2" type="revolute">
-        <origin xyz="0.4 0 ${arm_height}" rpy="0 0 0"/>
+        <origin xyz="${(scalex_1 * arm_dist_rot)} 0 ${arm_height}" rpy="0 0 0"/>
         <parent link="arm1"/>
         <child link="arm2"/>
@@ -41,5 +41,5 @@
         origon of joint set to ZERO, therefore controller input equals absolute z-position -->
     <joint name="joint_3" type="prismatic">
-    <origin xyz="0.25 0 ${-(base_height + arm_height)}" rpy="0 0 0"/>
+    <origin xyz="${(scalex_2 * arm_dist_rot)} 0 ${-(base_height + arm_height)}" rpy="0 0 0"/>
     <parent link="arm2"/>
     <child link="lin"/>
